Commit message: add child param to xacro
Signed-off-by: Paul Gesel <paulgesel@gmail.com>

File: descriptions/brackets/mtc_ur_tool_changer/mtc_ur_tool_changer.urdf.xacro (robot description, xacro)
@@ -1,8 +1,8 @@
 <?xml version="1.0" encoding="utf-8"?>
 <robot xmlns:xacro="http://ros.org/wiki/xacro">
-  <xacro:macro name="mtc_ur_tool_changer" params="prefix connected_to rotation:=^|${0.0}">
+  <xacro:macro name="mtc_ur_tool_changer" params="prefix parent child rotation:=^|${0.0}">
     <joint name="${prefix}tool_changer_joint" type="fixed">
       <!-- The parent link must be read from the robot model it is attached to. -->
-      <parent link="${connected_to}"/>
+      <parent link="${parent}"/>
       <child link="${prefix}tool_changer_link"/>
       <origin xyz="0 0 0" rpy="0 0 ${rotation}"/>
@@ -27,5 +27,5 @@
       <origin xyz="0 0 0.0331" rpy="0 0 0"/>
     </joint>
-    <link name="${prefix}tool_changer_tool0"/>
+    <link name="${child}"/>
   </xacro:macro>
 </robot>
