Commit message: add child parent as params
Signed-off-by: Paul Gesel <paulgesel@gmail.com>

File: descriptions/brackets/ur_realsense_camera_adapter/picknik_ur_camera_adapter.urdf.xacro (robot description, xacro)
@@ -1,8 +1,8 @@
 <?xml version="1.0" encoding="utf-8"?>
 <robot xmlns:xacro="http://ros.org/wiki/xacro">
-  <xacro:macro name="ur_realsense_camera_adapter" params="prefix connected_to rotation:=^|${0.0} camera_mount_pitch_offset:=^|${6.0 * pi / 180}">
+  <xacro:macro name="ur_realsense_camera_adapter" params="prefix parent child_camera child_tool rotation:=^|${0.0} camera_mount_pitch_offset:=^|${6.0 * pi / 180}">
     <joint name="${prefix}realsense_camera_adapter_joint" type="fixed">
       <!-- The parent link must be read from the robot model it is attached to. -->
-      <parent link="${connected_to}"/>
+      <parent link="${parent}"/>
       <child link="${prefix}realsense_camera_adapter_link"/>
       <origin xyz="0 0 0" rpy="0 0 ${rotation}"/>
@@ -25,11 +25,11 @@
     <joint name="${prefix}realsense_camera_adapter_tool0_joint" type="fixed">
       <parent link="${prefix}realsense_camera_adapter_link"/>
-      <child link="${prefix}realsense_camera_adapter_tool0"/>
+      <child link="${child_tool}"/>
       <origin xyz="0 0 0.007" rpy="0 0 0"/>
     </joint>
-    <link name="${prefix}d415_mount_link"/>
+    <link name="${child_camera}"/>
     <joint name="${prefix}d415_mount_joint" type="fixed">
       <parent link="${prefix}realsense_camera_adapter_link"/>
-      <child link="${prefix}d415_mount_link"/>
+      <child link="${child_camera}"/>
       <origin xyz="0 -0.067 0.0171" rpy="0 ${-pi/2 + camera_mount_pitch_offset} ${pi/2}"/>
     </joint>

Commit message: Changed STL and Renamed Link
Used picknik_ur5_realsense_camera_adapter_rev2_collision.stl from another branch main had the wrong format.

File: descriptions/brackets/ur_realsense_camera_adapter/picknik_ur_camera_adapter.urdf.xacro (robot description, xacro)
@@ -22,5 +22,5 @@
         </collision>
     </link>
-    <link name="${prefix}realsense_camera_adapter_tool0"/>
+    <link name="${child_tool}"/>
     <joint name="${prefix}realsense_camera_adapter_tool0_joint" type="fixed">
       <parent link="${prefix}realsense_camera_adapter_link"/>
